File: front-panel/schematics/ci_vfd.sch (KiCad schematic (older format))
At the start: 66 parts, among them J1 CONN_01X11, J3 CONN_02X06, Q1 Q_NPN_BCE, SW1 Menu, SW2 Right, SW3 Down, SW4 Up, SW5 Ok, SW6 Left, SW7 Back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

Commit message: Schematic: renamed SPI wires
Connections:
- net AT26: no longer C35.1, E2.2, R17.2
- net AT14 renamed /SS
- net AT15 renamed MOSI
- net AT16 renamed MISO
- net AT17 renamed SCK
- new net REQ: C35.1, E2.2, R17.2
Changed lines of the file:
@@
 EESchema Schematic File Version 2
-LIBS:power
-LIBS:device
-LIBS:transistors
-LIBS:conn
-LIBS:linear
-LIBS:regul
-LIBS:74xx
-LIBS:cmos4000
-LIBS:adc-dac
-LIBS:memory
-LIBS:xilinx
-LIBS:microcontrollers
-LIBS:dsp
-LIBS:microchip
-LIBS:analog_switches
-LIBS:motorola
-LIBS:texas
-LIBS:intel
-LIBS:audio
-LIBS:interface
-LIBS:digital-audio
-LIBS:philips
-LIBS:display
-LIBS:cypress
-LIBS:siliconi
-LIBS:opto
-LIBS:atmel
-LIBS:contrib
-LIBS:valves
 LIBS:TSOP38238
 LIBS:ci_vfd-cache
@@
 AVCC
 Text Label 4050 5200 2    60   ~ 0
-AT26
+REQ
 Text Label 3150 1900 2    60   ~ 0
 AT26
@@
 KM2
 Text Label 1850 7050 2    60   ~ 0
-AT16
+MISO
 Text Label 5900 1800 0    60   ~ 0
 KM3
@@
 $EndComp
 Text Label 2400 6200 2    60   ~ 0
-AT15
+MOSI
 Text Label 3300 7600 1    60   ~ 0
 Orange
@@
 $EndComp
 Text Label 2400 5050 2    60   ~ 0
-AT17
+SCK
 $Comp
 L R R2
@@
 $EndComp
 Text Label 2400 3900 2    60   ~ 0
-AT14
+/SS
 Text Label 3100 7600 1    60   ~ 0
 Brown
@@
 $EndComp
 Text Label 3150 1250 2    60   ~ 0
-AT17
+SCK
 Text Label 3150 1150 2    60   ~ 0
-AT16
+MISO
 Text Label 3150 1050 2    60   ~ 0
-AT15
+MOSI
 Text Label 3150 950  2    60   ~ 0
-AT14
+/SS
 $Comp
 L TSOP38238 U3
@@
 	7500 4250 7500 4600
 Text Label 7500 4600 1    60   ~ 0
-AT14
+/SS
 Wire Wire Line
 	7300 3750 7300 3400
 Text Label 7300 3400 3    60   ~ 0
-AT15
+MOSI
 Wire Wire Line
 	7200 4250 7200 4600
 Text Label 7200 4600 1    60   ~ 0
-AT16
+MISO
 Wire Wire Line
 	7300 4250 7300 4600
 Text Label 7300 4600 1    60   ~ 0
-AT17
+SCK
 Wire Wire Line
 	7400 4250 7400 4600
